File: PCBs/PCBs.kicad_sch (KiCad schematic)
At the start: 2 parts, among them U2 74HC595

Commit message: pcb
Parts:
- added J1, J2, J3, J4: Conn_01x50_Pin, Connector_FFC-FPC:Molex_54132-5033_1x50-1MP_P0.5mm_Horizontal, symbol Connector:Conn_01x50_Pin
- added U10, U11, U12, U13, U14, U15, U16, U17, U18, U19, U20, U21, U22, U23, U24, U25, U26, U27, U28, U29, U3, U30, U31, U32, U33, U34, U35, U36, U37, U38, U39, U4, U40, U5, U6, U7, U8, U9: ~, MyLib:K1HT661A-FTPRNT, symbol MyLib:K1HT661A-SMBL
- added U41, U42, U43, U44, U45, U46, U47, U48, U49, U50, U51, U52, U53, U54, U55, U56, U57, U58, U59, U60, U61, U62, U63, U64, U65, U66, U67, U68, U69, U70, U71, U72, U73, U74, U75, U76, U77, U78, U79, U80, U81, U82, U83, U84, U85, U86, U87, U88: ~, MyLib:BF422-FTPRNT, symbol MyLib:BF422
Connections:
- no-connect marks 0 -> 76
Other:
- company: (none) -> Astrolate
- title: (none) -> MC6205-1
- moved on the sheet: U1, U2
