File: Power-PCB/Power-PCB.kicad_pcb (KiCad board)
At the start: 2 copper layers, 139.1 x 139.1 mm, 192 parts, among them J1 Conn_01x50_Pin, J2 Conn_01x50_Pin, J3 Conn_01x50_Pin, J4 Conn_01x50_Pin

Commit message: pcb updates
Parts:
- added U1: ~, MyLibFtprnt:BF422-FTPRNT, B.Cu at (51.1, 57.4)
- added U15: ~, MyLibFtprnt:BF422-FTPRNT, B.Cu at (62.2, 85.4)
- added U16: ~, MyLibFtprnt:BF422-FTPRNT, B.Cu at (51.0, 87.4)
- added U17: ~, MyLibFtprnt:BF422-FTPRNT, B.Cu at (56.6, 89.4)
- added U18: ~, MyLibFtprnt:BF422-FTPRNT, B.Cu at (62.1, 91.4)
- added U19: ~, MyLibFtprnt:BF422-FTPRNT, B.Cu at (51.1, 93.4)
- added U2: ~, MyLibFtprnt:BF422-FTPRNT, B.Cu at (56.6, 59.4)
- added U20: ~, MyLibFtprnt:BF422-FTPRNT, B.Cu at (56.6, 95.4)
- added U21: ~, MyLibFtprnt:BF422-FTPRNT, B.Cu at (62.2, 97.4)
- added U22: ~, MyLibFtprnt:BF422-FTPRNT, B.Cu at (51.1, 99.4)
- added U23: ~, MyLibFtprnt:BF422-FTPRNT, B.Cu at (56.6, 101.4)
- added U24: ~, MyLibFtprnt:BF422-FTPRNT, B.Cu at (62.2, 103.4)
- added U25: ~, MyLibFtprnt:BF422-FTPRNT, B.Cu at (51.1, 105.4)
- added U26: ~, MyLibFtprnt:BF422-FTPRNT, B.Cu at (56.6, 107.4)
- added U27: ~, MyLibFtprnt:BF422-FTPRNT, B.Cu at (62.1, 109.4)
- added U28: ~, MyLibFtprnt:BF422-FTPRNT, B.Cu at (51.1, 111.4)
- added U29: ~, MyLibFtprnt:BF422-FTPRNT, B.Cu at (56.6, 113.4)
- added U3: ~, MyLibFtprnt:BF422-FTPRNT, B.Cu at (62.2, 61.4)
- added U30: ~, MyLibFtprnt:BF422-FTPRNT, B.Cu at (62.1, 115.4)
- added U31: ~, MyLibFtprnt:BF422-FTPRNT, B.Cu at (51.1, 117.4)
- added U32: ~, MyLibFtprnt:BF422-FTPRNT, B.Cu at (56.6, 119.4)
- added U33: ~, MyLibFtprnt:BF422-FTPRNT, B.Cu at (62.2, 121.4)
- added U34: ~, MyLibFtprnt:BF422-FTPRNT, B.Cu at (51.1, 123.4)
- added U35: ~, MyLibFtprnt:BF422-FTPRNT, B.Cu at (56.6, 125.4)
- added U36: ~, MyLibFtprnt:BF422-FTPRNT, B.Cu at (62.1, 127.4)
- added U37: ~, MyLibFtprnt:BF422-FTPRNT, B.Cu at (51.1, 129.4)
- added U38: ~, MyLibFtprnt:BF422-FTPRNT, B.Cu at (56.6, 131.4)
- added U39: ~, MyLibFtprnt:BF422-FTPRNT, B.Cu at (62.2, 133.4)
- added U4: ~, MyLibFtprnt:BF422-FTPRNT, B.Cu at (51.1, 63.4)
- added U40: ~, MyLibFtprnt:BF422-FTPRNT, B.Cu at (44.3, 149.6)
- U10, U11, U12, U13, U14, U5, U6, U7, U8, U9: footprint MyLib:K1HT661A-FTPRNT -> MyLibFtprnt:BF422-FTPRNT
- moved U7 49.9 mm to (51.1, 69.4), turned to 0 degrees
- moved U14 44.7 mm to (56.6, 83.4), turned to 0 degrees
- moved U6 43.5 mm to (62.1, 67.5), turned to 0 degrees
- moved U13 25.8 mm to (51.1, 81.4), turned to 0 degrees
- moved U11 24.9 mm to (56.6, 77.4), turned to 0 degrees
- moved U5 19.6 mm to (56.6, 65.4), turned to 0 degrees
- moved U41 17.5 mm to (48.2, 29.9)
- moved U42 16.0 mm to (48.3, 43.5), turned to -90 degrees
- moved U9 14.7 mm to (62.2, 73.4), turned to 0 degrees
- moved U12 14.5 mm to (62.2, 79.4), turned to 0 degrees
- moved U10 13.1 mm to (51.1, 75.4), turned to 0 degrees
- moved U8 8.71 mm to (56.6, 71.4), turned to 0 degrees
- moved U74 5.73 mm to (150.7, 136.5)
- moved U100 5.73 mm to (150.7, 100.5)
- moved U101 5.73 mm to (145.2, 102.5)
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- renumbered J4 to J1, J1 to J3, J3 to J4, U71 to U100, U72 to U101, U73 to U102, U74 to U103, U75 to U104, U76 to U105, U77 to U106, U78 to U107, U79 to U108, U80 to U109, U81 to U110, U82 to U111, U83 to U112, U84 to U113, U85 to U114, U86 to U115, U56 to U116, U57 to U117, U3 to U41, U4 to U42, U61 to U43, U60 to U44, U18 to U45, U19 to U46, U20 to U47, U28 to U48, U29 to U49, U30 to U50, U59 to U51, U88 to U52, U23 to U53, U24 to U54, U25 to U55, U33 to U56, U34 to U57, U35 to U58, U1 to U59, U87 to U60, U38 to U61, U39 to U62, U31 to U63, U15 to U64, U16 to U65, U21 to U66, U58 to U67, U36 to U68, U37 to U69, U32 to U70, U26 to U71, U27 to U72, U22 to U73, U54 to U74, U55 to U75, U17 to U76, U40 to U77, U41 to U78, U42 to U79, U43 to U80, U44 to U81, U45 to U82, U46 to U83, U47 to U84, U48 to U85, U49 to U86, U50 to U87, U51 to U88, U52 to U89, U53 to U90, U62 to U91, U63 to U92, U64 to U93, U65 to U94, U66 to U95, U67 to U96, U68 to U97, U69 to U98, U70 to U99
Connections:
- U10 pad 1: unconnected-(U10-Free-Pad1) -> /PA83
- U10 pad 2: /PA22 -> +250V
- U10 pad 3: /PA79 -> /СPA83
- U11 pad 1: unconnected-(U11-Free-Pad1) -> /PA20
- U11 pad 2: /PA26 -> +250V
- U11 pad 3: /PA75 -> /СPA20
- U12 pad 1: unconnected-(U12-Free-Pad1) -> /PA81
- U12 pad 2: /PA30 -> +250V
- U12 pad 3: /PA71 -> /СPA81
- U13 pad 1: unconnected-(U13-Free-Pad1) -> /PA22
- U13 pad 2: /PA34 -> +250V
- U13 pad 3: /PA67 -> /СPA22
- U14 pad 1: unconnected-(U14-Free-Pad1) -> /PA79
- U14 pad 2: /PA46 -> +250V
- U14 pad 3: /PA55 -> /СPA79
- U5 pad 1: unconnected-(U5-Free-Pad1) -> /PA14
- U5 pad 2: /PA10 -> +250V
- U5 pad 3: /PA91 -> /СPA14
- U6 pad 1: unconnected-(U6-Free-Pad1) -> /PA87
- U6 pad 2: /PA38 -> +250V
- U6 pad 3: /PA63 -> /СPA87
- U7 pad 1: unconnected-(U7-Free-Pad1) -> /PA16
- U7 pad 2: /PA42 -> +250V
- U7 pad 3: /PA59 -> /СPA16
- U8 pad 1: unconnected-(U8-Free-Pad1) -> /PA85
- U8 pad 2: /PA14 -> +250V
- U8 pad 3: /PA87 -> /СPA85
- U9 pad 1: unconnected-(U9-Free-Pad1) -> /PA18
- U9 pad 2: /PA18 -> +250V
- U9 pad 3: /PA83 -> /СPA18
Routing:
- net /CPA80: track 213.7 -> 62.2 mm, vias 1 -> 0
- net /CPA21: track 206.8 -> 66.2 mm, vias 1 -> 0
- net /CPA25: track 207.8 -> 68.5 mm, vias 1 -> 0
- net /CPA78: track 200.2 -> 72.5 mm, vias 1 -> 0
- net +250V: track 877.5 -> 752.9 mm, vias 23 -> 1
- net /СPA57: track 73.4 -> 29.1 mm, vias 2 -> 1
- net /PA94: track 40.1 -> 4.89 mm, vias 2 -> 0
- net /СPA44: track 60.5 -> 29.3 mm, vias 2 -> 1
- net /PA53: track 30.8 -> 3.95 mm
- net /PA83: track 27.9 -> 2.66 mm
- net /PA10: track 25.3 -> 2.65 mm
- net /PA7: track 27.9 -> 6.37 mm
- net /СPA48: track 29.0 -> 50.3 mm
- net /PA38: track 29.2 -> 8.19 mm
- net /СPA93: track 104.4 -> 125.4 mm, vias 2 -> 0
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Other:
- board size 139.1 x 139.1 mm -> 139 x 139 mm
- board text added: "GIP-1000"
