File: Power-PCB/Power-PCB.kicad_sch (KiCad schematic)
At the start: 192 parts, among them J1 Conn_01x50_Pin, J2 Conn_01x50_Pin, J3 Conn_01x50_Pin, J4 Conn_01x50_Pin, U2 74HC595

Commit message: pcb updates
Parts:
- removed U10, U11, U12, U13, U14, U5, U6, U7, U8, U9: ~, MyLib:K1HT661A-FTPRNT, symbol MyLib:K1HT661A-SMBL
- removed U2: 74HC595, Package_DIP:DIP-16_W7.62mm, symbol 74xx:74HC595
- added U1, U10, U11, U12, U13, U14, U15, U16, U17, U18, U19, U2, U20, U21, U22, U23, U24, U25, U26, U27, U28, U29, U3, U30, U31, U32, U33, U34, U35, U36, U37, U38, U39, U4, U40, U5, U6, U7, U8, U9: ~, MyLibFtprnt:BF422-FTPRNT, symbol MyLib:BF422
- renumbered J4 to J1, J1 to J3, J3 to J4, U71 to U100, U72 to U101, U73 to U102, U74 to U103, U75 to U104, U76 to U105, U77 to U106, U78 to U107, U79 to U108, U80 to U109, U81 to U110, U82 to U111, U83 to U112, U84 to U113, U85 to U114, U86 to U115, U56 to U116, U57 to U117, U3 to U41, U4 to U42, U61 to U43, U60 to U44, U18 to U45, U19 to U46, U20 to U47, U28 to U48, U29 to U49, U30 to U50, U59 to U51, U88 to U52, U23 to U53, U24 to U54, U25 to U55, U33 to U56, U34 to U57, U35 to U58, U1 to U59, U87 to U60, U38 to U61, U39 to U62, U31 to U63, U15 to U64, U16 to U65, U21 to U66, U58 to U67, U36 to U68, U37 to U69, U32 to U70, U26 to U71, U27 to U72, U22 to U73, U54 to U74, U55 to U75, U17 to U76, U40 to U77, U41 to U78, U42 to U79, U43 to U80, U44 to U81, U45 to U82, U46 to U83, U47 to U84, U48 to U85, U49 to U86, U50 to U87, U51 to U88, U52 to U89, U53 to U90, U62 to U91, U63 to U92, U64 to U93, U65 to U94, U66 to U95, U67 to U96, U68 to U97, U69 to U98, U70 to U99
Connections:
- net +250V: now also U1.2 (C), U10.2 (C), U11.2 (C), U12.2 (C), U13.2 (C), U14.2 (C), U15.2 (C), U16.2 (C), U17.2 (C), U18.2 (C), U19.2 (C), U2.2 (C), U20.2 (C), U21.2 (C), U22.2 (C), U23.2 (C), U24.2 (C), U25.2 (C), U26.2 (C), U27.2 (C), U28.2 (C), U29.2 (C), U3.2 (C), U30.2 (C), U31.2 (C), U32.2 (C), U33.2 (C), U34.2 (C), U35.2 (C), U36.2 (C), U37.2 (C), U38.2 (C), U39.2 (C), U4.2 (C), U40.2 (C), U5.2 (C), U6.2 (C), U7.2 (C), U8.2 (C), U9.2 (C)
- net PA10: now also U1.1 (E)
- net PA12: now also U3.1 (E)
- net PA14: now also U5.1 (E)
- net PA16: now also U7.1 (E)
- net PA18: now also U9.1 (E)
- net PA20: now also U11.1 (E)
- net PA22: now also U13.1 (E)
- net PA24: now also U15.1 (E)
- net PA26: now also U17.1 (E)
- net PA28: now also U19.1 (E)
- net PA30: now also U21.1 (E)
- net PA32: now also U23.1 (E)
- net PA34: now also U25.1 (E)
- net PA36: now also U27.1 (E)
- net PA38: now also U29.1 (E)
- net PA40: now also U31.1 (E)
- net PA42: now also U33.1 (E)
- net PA44: now also U35.1 (E)
- net PA46: now also U37.1 (E)
- net PA48: now also U39.1 (E)
- net PA53: now also U40.1 (E)
- net PA55: now also U38.1 (E)
- net PA57: now also U36.1 (E)
- net PA59: now also U34.1 (E)
- net PA61: now also U32.1 (E)
- net PA63: now also U30.1 (E)
- net PA65: now also U28.1 (E)
- net PA67: now also U26.1 (E)
- net PA69: now also U24.1 (E)
- net PA71: now also U22.1 (E)
- net PA73: now also U20.1 (E)
- net PA75: now also U18.1 (E)
- net PA77: now also U16.1 (E)
- net PA79: now also U14.1 (E)
- net PA81: now also U12.1 (E)
- net PA83: now also U10.1 (E)
- net PA85: now also U8.1 (E)
- net PA87: now also U6.1 (E)
- net PA89: now also U4.1 (E)
- net PA91: now also U2.1 (E)
- net СPA10: now also U1.3 (B)
- net СPA12: now also U3.3 (B)
- net СPA14: now also U5.3 (B)
- net СPA16: now also U7.3 (B)
- net СPA18: now also U9.3 (B)
- net СPA20: now also U11.3 (B)
- net СPA22: now also U13.3 (B)
- net СPA24: now also U15.3 (B)
- net СPA26: now also U17.3 (B)
- net СPA28: now also U19.3 (B)
- net СPA30: now also U21.3 (B)
- net СPA32: now also U23.3 (B)
- net СPA34: now also U25.3 (B)
- net СPA36: now also U27.3 (B)
- net СPA38: now also U29.3 (B)
- net СPA40: now also U31.3 (B)
- net СPA42: now also U33.3 (B)
- net СPA44: now also U35.3 (B)
- net СPA46: now also U37.3 (B)
- net СPA48: now also U39.3 (B)
- net СPA53: now also U40.3 (B)
- net СPA55: now also U38.3 (B)
- net СPA57: now also U36.3 (B)
- net СPA59: now also U34.3 (B)
- net СPA61: now also U32.3 (B)
- net СPA63: now also U30.3 (B)
- net СPA65: now also U28.3 (B)
- net СPA67: now also U26.3 (B)
- net СPA69: now also U24.3 (B)
- net СPA71: now also U22.3 (B)
- net СPA73: now also U20.3 (B)
- net СPA75: now also U18.3 (B)
- net СPA77: now also U16.3 (B)
- net СPA79: now also U14.3 (B)
- net СPA81: now also U12.3 (B)
- net СPA83: now also U10.3 (B)
- net СPA85: now also U8.3 (B)
- net СPA87: now also U6.3 (B)
- net СPA89: now also U4.3 (B)
- net СPA91: now also U2.3 (B)
- no-connect marks 76 -> 56
Other:
- moved on the sheet: R1, R10, R100, R11, R12, R13, R14, R15, R16, R17, R18, R19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
